File: Hardware/Without_Regulator/dps5005control.sch (KiCad schematic (older format))
At the start: 10 parts, among them P2 CONN_4, P3 CONN_5X2, P4 CONN_7, U2 ATTINY2313-20PU

Commit message: HARD: Migrated the version without regulator to the new kicad symbol table.
Parts:
- removed C1: 100u, w_capacitors:CP_6.3x11mm, symbol CP1_Small
- removed D1, D2: LED_Small_ALT, LEDs:LED_D5.0mm, symbol LED_Small_ALT
- removed U2: ATTINY2313-20PU, w_pth_circuits:dil_20-300_socket, symbol ATTINY2313-20PU
- added C1: 100 uF, w_capacitors:CP_6.3x11mm, symbol device:CP1_Small
- added D1, D2: LED_Small_ALT, symbol device:LED_Small_ALT
- added U2: ATTINY2313-20PU, symbol atmel:ATTINY2313-20PU
- P2: symbol CONN_4 -> conn:CONN_4
- P3: symbol CONN_5X2 -> conn:CONN_5X2
- P4: symbol CONN_7 -> conn:CONN_7
- R1, R2, R3: symbol R -> w_device:R
Changed lines of the file:
@@
-EESchema Schematic File Version 3
-LIBS:power
-LIBS:device
-LIBS:transistors
-LIBS:conn
-LIBS:linear
-LIBS:regul
-LIBS:74xx
-LIBS:cmos4000
-LIBS:adc-dac
-LIBS:memory
-LIBS:xilinx
-LIBS:microcontrollers
-LIBS:dsp
-LIBS:microchip
-LIBS:analog_switches
-LIBS:motorola
-LIBS:texas
-LIBS:intel
-LIBS:audio
-LIBS:interface
-LIBS:digital-audio
-LIBS:philips
-LIBS:display
-LIBS:cypress
-LIBS:siliconi
-LIBS:opto
-LIBS:atmel
-LIBS:contrib
-LIBS:valves
-LIBS:w_analog
-LIBS:w_connectors
-LIBS:w_device
-LIBS:w_logic
-LIBS:w_memory
-LIBS:w_microcontrollers
-LIBS:w_opto
-LIBS:w_relay
-LIBS:w_rtx
-LIBS:w_transistor
-LIBS:w_vacuum
+EESchema Schematic File Version 4
 LIBS:dps5005control-cache
 EELAYER 26 0
@@
 $EndDescr
 $Comp
-L ATTINY2313-20PU U2
-U 1 1 59ABC6E6
-P 3875 2350
-F 0 "U2" H 4025 3500 50  0000 C CNN
-F 1 "ATTINY2313-20PU" H 4325 3400 50  0000 C CNN
-F 2 "w_pth_circuits:dil_20-300_socket" H 3875 2350 50  0001 C CIN
-F 3 "" H 3875 2350 50  0001 C CNN
-	1    3875 2350
-	1    0    0    -1
-$EndComp
-$Comp
-L GND #PWR01
+L power:GND #PWR01
 U 1 1 59ABC7E4
 P 3875 3450
@@
 	3875 3450 3875 3350
 $Comp
-L CONN_4 P2
+L conn:CONN_4 P2
 U 1 1 59ABD3B5
 P 2175 2825
@@
 	5025 2550 5225 2550
 $Comp
-L CONN_5X2 P3
+L conn:CONN_5X2 P3
 U 1 1 59ABD882
 P 6650 3000
@@
 Connection ~ 7150 3000
 $Comp
-L GND #PWR06
+L power:GND #PWR06
 U 1 1 59ABDA21
 P 7150 3300
@@
 RST
 $Comp
-L R R1
+L w_device:R R1
 U 1 1 59ABE305
 P 3275 1150
@@
 CC_MODE
 $Comp
-L R R2
+L w_device:R R2
 U 1 1 59AC02EA
 P 1625 1600
@@
 $EndComp
 Wire Wire Line
-	1775 1600 1925 1600
-Wire Wire Line
-	1475 1600 1325 1600
+	1725 1600 1925 1600
+Wire Wire Line
+	1325 1600 1525 1600
 Text Label 1325 1600 2    60   ~ 0
 CC_MODE
 $Comp
-L GND #PWR011
+L power:GND #PWR011
 U 1 1 59AC07C6
 P 2275 1750
@@
 Wire Wire Line
 	2275 1600 2275 1750
-$Comp
-L LED_Small_ALT D1
-U 1 1 59AC0B63
-P 2025 1600
-F 0 "D1" H 2025 1835 50  0000 C CNN
-F 1 "LED_Small_ALT" H 2025 1744 50  0000 C CNN
-F 2 "LEDs:LED_D5.0mm" V 2025 1600 50  0001 C CNN
-F 3 "" V 2025 1600 50  0001 C CNN
-	1    2025 1600
-	-1   0    0    -1
-$EndComp
 Wire Wire Line
 	1825 2675 1725 2675
@@
 	1725 2975 1725 3075
 $Comp
-L GND #PWR012
+L power:GND #PWR012
 U 1 1 59AC0F5A
 P 1725 3075
@@
 NoConn ~ 5025 2650
 $Comp
-L R R3
+L w_device:R R3
 U 1 1 59AD66A9
 P 1625 2150
@@
 $EndComp
 Wire Wire Line
-	1775 2150 1925 2150
-Wire Wire Line
-	1025 2150 1475 2150
-$Comp
-L GND #PWR014
+	1725 2150 1925 2150
+Wire Wire Line
+	1025 2150 1525 2150
+$Comp
+L power:GND #PWR014
 U 1 1 59AD66B3
 P 2275 2300
@@
 	2275 2150 2275 2300
 $Comp
-L LED_Small_ALT D2
-U 1 1 59AD66BB
-P 2025 2150
-F 0 "D2" H 2025 2385 50  0000 C CNN
-F 1 "LED_Small_ALT" H 2025 2294 50  0000 C CNN
-F 2 "LEDs:LED_D5.0mm" V 2025 2150 50  0001 C CNN
-F 3 "" V 2025 2150 50  0001 C CNN
-	1    2025 2150
-	-1   0    0    -1
-$EndComp
-$Comp
-L CONN_7 P4
+L conn:CONN_7 P4
 U 1 1 59AE78AB
 P 6275 1825
@@
 ENC1_SW
 $Comp
-L GND #PWR015
+L power:GND #PWR015
 U 1 1 59AE7D7C
 P 6825 2325
@@
 	6825 2125 6825 2325
 $Comp
-L +3,3V #PWR02
+L power:+3,3V #PWR02
 U 1 1 59DA2C26
 P 1725 2575
@@
 	1325 2150 1325 2050
 $Comp
-L +3,3V #PWR03
+L power:+3,3V #PWR03
 U 1 1 59DA2D0C
 P 1325 2050
@@
 	7150 2800 7150 2700
 $Comp
-L +3,3V #PWR04
+L power:+3,3V #PWR04
 U 1 1 59DA2E6B
 P 7150 2700
@@
 $EndComp
 $Comp
-L +3,3V #PWR05
+L power:+3,3V #PWR05
 U 1 1 59DA3184
 P 3875 900
@@
 $EndComp
 $Comp
-L PWR_FLAG #FLG01
+L power:PWR_FLAG #FLG01
 U 1 1 59DA330D
 P 1025 2125
@@
 Connection ~ 1325 2150
 $Comp
-L PWR_FLAG #FLG02
+L power:PWR_FLAG #FLG02
 U 1 1 59DA35AC
 P 7400 3125
@@
 	7400 3200 7400 3125
 $Comp
-L CP1_Small C1
-U 1 1 59DA4007
-P 1175 2825
-F 0 "C1" H 1266 2871 50  0000 L CNN
-F 1 "100u" H 1266 2780 50  0000 L CNN
-F 2 "w_capacitors:CP_6.3x11mm" H 1175 2825 50  0001 C CNN
-F 3 "" H 1175 2825 50  0001 C CNN
-	1    1175 2825
-	1    0    0    -1
-$EndComp
-$Comp
-L GND #PWR08
+L power:GND #PWR08
 U 1 1 59DA420B
 P 1175 3075
@@
 $EndComp
 $Comp
-L +3,3V #PWR07
+L power:+3,3V #PWR07
 U 1 1 59DA422A
 P 1175 2575
@@
 	1175 2925 1175 3075
 Wire Wire Line
-	3425 1150 3875 1150
+	3375 1150 3875 1150
 Connection ~ 3875 1150
 Wire Wire Line
-	2675 1150 3125 1150
+	2675 1150 3175 1150
+$Comp
+L device:LED_Small_ALT D1
+U 1 1 5A0D5999
+P 2025 1600
+F 0 "D1" H 2025 1835 50  0000 C CNN
+F 1 "LED_Small_ALT" H 2025 1744 50  0000 C CNN
+F 2 "" V 2025 1600 50  0001 C CNN
+F 3 "" V 2025 1600 50  0001 C CNN
+	1    2025 1600
+	-1   0    0    -1
+$EndComp
+$Comp
+L device:LED_Small_ALT D2
+U 1 1 5A0D5AD4
+P 2025 2150
+F 0 "D2" H 2025 2385 50  0000 C CNN
+F 1 "LED_Small_ALT" H 2025 2294 50  0000 C CNN
+F 2 "" V 2025 2150 50  0001 C CNN
+F 3 "" V 2025 2150 50  0001 C CNN
+	1    2025 2150
+	-1   0    0    -1
+$EndComp
+$Comp
+L atmel:ATTINY2313-20PU U2
+U 1 1 5A0D5BF6
+P 3875 2350
+F 0 "U2" H 3875 2325 50  0000 C CNN
+F 1 "ATTINY2313-20PU" H 4350 3375 50  0000 C CNN
+F 2 "" H 3875 2350 50  0001 C CIN
+F 3 "http://www.atmel.com/Images/doc2543.pdf" H 3875 2350 50  0001 C CNN
+	1    3875 2350
+	1    0    0    -1
+$EndComp
+$Comp
+L device:CP1_Small C1
+U 1 1 5A0D6222
+P 1175 2825
+F 0 "C1" H 1266 2871 50  0000 L CNN
+F 1 "100 uF" H 1266 2780 50  0000 L CNN
+F 2 "w_capacitors:CP_6.3x11mm" H 1175 2825 50  0001 C CNN
+F 3 "" H 1175 2825 50  0001 C CNN
+	1    1175 2825
+	1    0    0    -1
+$EndComp
 $EndSCHEMATC
